Commit message: Add prefix param

File: control/gazebo_diff_drive_plugin.xacro (robot description, xacro)
@@ -1,17 +1,19 @@
 <?xml version="1.0"?>
 <robot xmlns:xacro="http://www.ros.org/wiki/xacro">
+  <!-- Define a macro with a prefix param for the Zed M camera description -->
+  <xacro:macro name="gazebo_diff_drive_plugin_description" params="prefix">
     <gazebo>
         <plugin name="gz::sim::systems::DiffDrive" filename="gz-sim-diff-drive-system">
-            <left_joint>front_left_wheel_joint</left_joint>
-            <right_joint>front_right_wheel_joint</right_joint>
-            <left_joint>back_left_wheel_joint</left_joint>
-            <right_joint>back_right_wheel_joint</right_joint>
+            <left_joint>${prefix}front_left_wheel_joint</left_joint>
+            <right_joint>${prefix}front_right_wheel_joint</right_joint>
+            <left_joint>${prefix}back_left_wheel_joint</left_joint>
+            <right_joint>${prefix}back_right_wheel_joint</right_joint>
             <wheel_separation>0.35</wheel_separation>
             <wheel_radius>0.08</wheel_radius>
             <max_linear_acceleration>0.033</max_linear_acceleration>
-            <topic>cmd_vel</topic>
-            <odom_topic>odom</odom_topic>
-            <frame_id>odom</frame_id>
-            <child_frame_id>base_link</child_frame_id>
+            <topic>${prefix}cmd_vel</topic>
+            <odom_topic>${prefix}odom</odom_topic>
+            <frame_id>${prefix}odom</frame_id>
+            <child_frame_id>${prefix}base_link</child_frame_id>
             <odom_publisher_frequency>30</odom_publisher_frequency>
             <tf_topic>/tf</tf_topic>
@@ -19,10 +21,11 @@
         <plugin filename="gz-sim-joint-state-publisher-system"
             name="gz::sim::systems::JointStatePublisher">
-            <topic>joint_states</topic>
-            <joint_name>front_left_wheel_joint</joint_name>
-            <joint_name>front_right_wheel_joint</joint_name>
-            <joint_name>back_left_wheel_joint</joint_name>
-            <joint_name>back_right_wheel_joint</joint_name>
+            <topic>${prefix}joint_states</topic>
+            <joint_name>${prefix}front_left_wheel_joint</joint_name>
+            <joint_name>${prefix}front_right_wheel_joint</joint_name>
+            <joint_name>${prefix}back_left_wheel_joint</joint_name>
+            <joint_name>${prefix}back_right_wheel_joint</joint_name>
         </plugin>
     </gazebo>
+  </xacro:macro>
 </robot>

Commit message: Refactor prefix handling

File: control/gazebo_diff_drive_plugin.xacro (robot description, xacro)
@@ -2,11 +2,18 @@
 <robot xmlns:xacro="http://www.ros.org/wiki/xacro">
   <!-- Define a macro with a prefix param for the Zed M camera description -->
-  <xacro:macro name="gazebo_diff_drive_plugin_description" params="prefix">
+  <xacro:macro name="gazebo_diff_drive_plugin_description" params="namespace prefix">
+    <!-- Properties -->
+    <xacro:if value="${prefix != ''}">
+      <xacro:property name="prefix_" value="${prefix}_"/>
+    </xacro:if>
+    <xacro:if value="${prefix == ''}">
+      <xacro:property name="prefix_" value=""/>
+    </xacro:if>
     <gazebo>
         <plugin name="gz::sim::systems::DiffDrive" filename="gz-sim-diff-drive-system">
-            <left_joint>${prefix}front_left_wheel_joint</left_joint>
-            <right_joint>${prefix}front_right_wheel_joint</right_joint>
-            <left_joint>${prefix}back_left_wheel_joint</left_joint>
-            <right_joint>${prefix}back_right_wheel_joint</right_joint>
+            <left_joint>${prefix_}front_left_wheel_joint</left_joint>
+            <right_joint>${prefix_}front_right_wheel_joint</right_joint>
+            <left_joint>${prefix_}back_left_wheel_joint</left_joint>
+            <right_joint>${prefix_}back_right_wheel_joint</right_joint>
             <wheel_separation>0.35</wheel_separation>
             <wheel_radius>0.08</wheel_radius>
@@ -15,5 +22,5 @@
             <odom_topic>odom</odom_topic>
             <frame_id>odom</frame_id>
-            <child_frame_id>${prefix}base_link</child_frame_id>
+            <child_frame_id>${prefix_}base_link</child_frame_id>
             <odom_publisher_frequency>30</odom_publisher_frequency>
             <tf_topic>/tf</tf_topic>
@@ -21,9 +28,9 @@
         <plugin filename="gz-sim-joint-state-publisher-system"
             name="gz::sim::systems::JointStatePublisher">
-            <topic>joint_states</topic>
-            <joint_name>${prefix}front_left_wheel_joint</joint_name>
-            <joint_name>${prefix}front_right_wheel_joint</joint_name>
-            <joint_name>${prefix}back_left_wheel_joint</joint_name>
-            <joint_name>${prefix}back_right_wheel_joint</joint_name>
+            <topic>$(arg namespace)/joint_states</topic>
+            <joint_name>${prefix_}front_left_wheel_joint</joint_name>
+            <joint_name>${prefix_}front_right_wheel_joint</joint_name>
+            <joint_name>${prefix_}back_left_wheel_joint</joint_name>
+            <joint_name>${prefix_}back_right_wheel_joint</joint_name>
         </plugin>
     </gazebo>

File: control/gazebo_ros2_control_plugin.xacro (robot description, xacro)
@@ -1,10 +1,17 @@
 <?xml version="1.0"?>
 <robot xmlns:xacro="http://www.ros.org/wiki/xacro">
-    <xacro:macro name="gazebo_ros2_control_plugin_description" params="prefix">
+    <xacro:macro name="gazebo_ros2_control_plugin_description" params="namespace prefix">
+        <!-- Properties -->
+        <xacro:if value="${prefix != ''}">
+            <xacro:property name="prefix_" value="${prefix}_"/>
+        </xacro:if>
+        <xacro:if value="${prefix == ''}">
+            <xacro:property name="prefix_" value=""/>
+        </xacro:if>
         <ros2_control name="GazeboSimSystem" type="system">
             <hardware>
                 <plugin>gz_ros2_control/GazeboSimSystem</plugin>
             </hardware>
-            <joint name="front_left_wheel_joint">
+            <joint name="${prefix_}front_left_wheel_joint">
                 <param name="id">3</param>
                 <command_interface name="velocity">
@@ -15,5 +22,5 @@
                 <state_interface name="velocity" />
             </joint>
-            <joint name="front_right_wheel_joint">
+            <joint name="${prefix_}front_right_wheel_joint">
                 <param name="id">4</param>
                 <command_interface name="velocity">
@@ -24,5 +31,5 @@
                 <state_interface name="position" />
             </joint>
-            <joint name="back_left_wheel_joint">
+            <joint name="${prefix_}back_left_wheel_joint">
                 <param name="id">1</param>
                 <command_interface name="velocity">
@@ -33,5 +40,5 @@
                 <state_interface name="velocity" />
             </joint>
-            <joint name="back_right_wheel_joint">
+            <joint name="${prefix_}back_right_wheel_joint">
                 <param name="id">2</param>
                 <command_interface name="velocity">
@@ -44,4 +51,9 @@
         </ros2_control>
         <gazebo>
+            <xacro:if value="${namespace != ''}">
+            <ros>
+                <namespace>$(arg namespace)</namespace>
+            </ros>
+            </xacro:if>
             <plugin name="gz_ros2_control::GazeboSimROS2ControlPlugin" filename="gz_ros2_control-system">
                 <parameters>$(find arcs_cohort_gazebo_sim)/config/ros2_control_params.yaml</parameters>
