Commit message: Refactor ros2_control params template generation

File: control/gazebo_ros2_control_plugin.xacro (robot description, xacro)
@@ -1,5 +1,5 @@
 <?xml version="1.0"?>
 <robot xmlns:xacro="http://www.ros.org/wiki/xacro">
-    <xacro:macro name="gazebo_ros2_control_plugin_description" params="namespace prefix">
+    <xacro:macro name="gazebo_ros2_control_plugin_description" params="namespace prefix ros2_control_params">
         <!-- Properties -->
         <xacro:if value="${prefix != ''}">
@@ -59,5 +59,5 @@
                 </ros>
                 </xacro:if>
-                <parameters>$(find arcs_cohort_gazebo_sim)/config/gazebo_ros2_control_params.yaml</parameters>
+                <parameters>$(arg ros2_control_params)</parameters>
             </plugin>
         </gazebo>

File: description/robot.gazebo.xacro (robot description, xacro)
@@ -6,6 +6,7 @@
     <xacro:arg name="camera_model" default="zedm" />
     <xacro:arg name="camera_resolution" default="VGA" />
+    <xacro:arg name="lidar_update_rate" default="10" />
+    <xacro:arg name="ros2_control_params" default="" />
     <xacro:arg name="use_lidar" default="false" />
-    <xacro:arg name="lidar_update_rate" default="10" />
     <xacro:arg name="use_ros2_control" default="false" />
     <!-- Include Gazebo files -->
@@ -31,5 +32,5 @@
     <!-- Conditionally call the appropriate Gazebo plugin description -->
     <xacro:if value="$(arg use_ros2_control)">
-        <xacro:gazebo_ros2_control_plugin_description namespace="$(arg namespace)" prefix="$(arg prefix)"/>
+        <xacro:gazebo_ros2_control_plugin_description namespace="$(arg namespace)" prefix="$(arg prefix)" ros2_control_params="$(arg ros2_control_params)"/>
     </xacro:if>
     <xacro:unless value="$(arg use_ros2_control)">
