Commit message: Add lunar terrain

File: description/lidar.gazebo.xacro (robot description, xacro)
@@ -2,5 +2,5 @@
 <robot xmlns:xacro="http://www.ros.org/wiki/xacro" name="robot">
     <xacro:property name="PI" value="3.1415926535897931" />
-    <xacro:macro name="lidar_description_gazebo" params="prefix lidar_update_rate=30">
+    <xacro:macro name="lidar_description_gazebo" params="prefix lidar_update_rate=10">
         <!-- LiDAR Gazebo -->
         <gazebo reference="${prefix}laser_frame">

File: description/robot.gazebo.xacro (robot description, xacro)
@@ -6,5 +6,5 @@
     <xacro:arg name="camera_resolution" default="HD720" />
     <xacro:arg name="use_lidar" default="false" />
-    <xacro:arg name="lidar_update_rate" default="30" />
+    <xacro:arg name="lidar_update_rate" default="10" />
     <xacro:arg name="use_ros2_control" default="false" />
     <!-- Include Gazebo files -->
